Commit message: Added proper xacro's for dslam boards

File: gopherturtle_description/robots/kobuki_hexagons_dslam_boards.urdf.xacro (robot description, xacro)
@@ -8,5 +8,7 @@
   <xacro:include filename="$(find gopherturtle_description)/urdf/turtlebot_library.urdf.xacro" />
   <kobuki/>
-  <stack_hexagons parent="base_link"/>
-  <dslam_boards  parent="base_link"/>
+  <stack_hexagons          parent="base_link"/>
+  <front_dslam_board       parent="base_link"/>
+  <back_dslam_board        parent="base_link"/>
+  <sensor_asus_xtion_pro   parent="base_link"/>
 </robot>

File: gopherturtle_description/urdf/sensors/dslam_boards.urdf.xacro (robot description, xacro)
@@ -21,5 +21,5 @@
         <!--This is for the left camera on the front DSLAM board-->
         <joint name="front_camera_left_joint" type="fixed">
-            <origin xyz="0 -50 0" rpy="0 0 0"/>
+            <origin xyz="0 -0.05 0" rpy="-1.57079633 0 1.57079633"/>
             <parent link="front_dslam_board_frame"/>
             <child link="front_camera_left_joint"/>
@@ -48,5 +48,5 @@
         <!--This is for the right camera on the front DSLAM board-->
         <joint name="front_camera_right_joint" type="fixed">
-            <origin xyz="0 50 0" rpy="0 0 0"/>
+            <origin xyz="0 0.05 0" rpy="-1.57079633 0 1.57079633"/>
             <parent link="front_dslam_board_frame"/>
             <child link="front_camera_right_joint"/>
@@ -92,5 +92,5 @@
         <!--This is for the left camera on the back DSLAM board-->
         <joint name="back_camera_left_joint" type="fixed">
-            <origin xyz="0 -50 0" rpy="0 0 0"/>
+            <origin xyz="0 -0.05 0" rpy="-1.57079633 0 1.57079633"/>
             <parent link="back_dslam_board_frame"/>
             <child link="back_camera_left_joint"/>
@@ -119,5 +119,5 @@
         <!--This is for the right camera on the front DSLAM board-->
         <joint name="back_camera_right_joint" type="fixed">
-            <origin xyz="0 50 0" rpy="0 0 0"/>
+            <origin xyz="0 0.05 0" rpy="-1.57079633 0 1.57079633"/>
             <parent link="back_dslam_board_frame"/>
             <child link="back_camera_right_joint"/>
@@ -144,6 +144,97 @@
             </inertial>
         </link>
-        <!--Kinect sensor for simulation-->
-        <turtlebot_sim_3dsensor/>
     </xacro:macro>
+    <!-- Xacro properties -->
+  <xacro:property name="M_SCALE" value="0.001"/>
+  <xacro:property name="asus_xtion_pro_depth_rel_rgb_py" value="0.0270" />
+  <xacro:property name="asus_xtion_pro_cam_rel_rgb_py"   value="-0.0220" />
+  <!-- Parameterised in part by the values in turtlebot_properties.urdf.xacro -->
+  <xacro:macro name="sensor_asus_xtion_pro" params="parent">
+    <joint name="camera_rgb_joint" type="fixed">
+      <origin xyz="${cam_px} ${cam_py} ${cam_pz}"
+              rpy="${cam_or} ${cam_op} ${cam_oy}"/>
+      <parent link="${parent}"/>
+      <child link="camera_rgb_frame" />
+    </joint>
+    <link name="camera_rgb_frame">
+      <inertial>
+        <mass value="0.001" />
+        <origin xyz="0 0 0" />
+        <inertia ixx="0.0001" ixy="0.0" ixz="0.0"
+          iyy="0.0001" iyz="0.0"
+          izz="0.0001" />
+      </inertial>
+    </link>
+    <joint name="camera_rgb_optical_joint" type="fixed">
+      <origin xyz="0 0 0" rpy="${-M_PI/2} 0 ${-M_PI/2}" />
+      <parent link="camera_rgb_frame" />
+      <child link="camera_rgb_optical_frame" />
+    </joint>
+    <link name="camera_rgb_optical_frame">
+      <inertial>
+        <mass value="0.001" />
+        <origin xyz="0 0 0" />
+        <inertia ixx="0.0001" ixy="0.0" ixz="0.0"
+          iyy="0.0001" iyz="0.0"
+          izz="0.0001" />
+      </inertial>
+    </link>
+    <joint name="camera_joint" type="fixed">
+      <origin xyz="0 ${asus_xtion_pro_cam_rel_rgb_py} 0"
+              rpy="0 0 0"/>
+      <parent link="camera_rgb_frame"/>
+      <child link="camera_link"/>
+    </joint>
+    <link name="camera_link">
+      <visual>
+        <origin xyz="-0.01 0 0" rpy="${-M_PI/2} -${M_PI} ${-M_PI/2}"/>
+        <geometry>
+          <mesh filename="package://gopherturtle_description/meshes/sensors/asus_xtion_pro_live.dae" scale="${M_SCALE} ${M_SCALE} ${M_SCALE}"/>
+        </geometry>
+      </visual>
+      <collision>
+        <origin xyz="0.0 0.0 0.0" rpy="0 0 0" />
+        <geometry>
+        <box size="0.0730 .2760 0.0720"/>
+      </geometry>
+      </collision>
+      <inertial>
+        <mass value="0.01" />
+        <origin xyz="0 0 0" />
+        <inertia ixx="0.001" ixy="0.0" ixz="0.0"
+          iyy="0.001" iyz="0.0"
+          izz="0.001" />
+      </inertial>
+    </link>
+    <joint name="camera_depth_joint" type="fixed">
+      <origin xyz="0 ${asus_xtion_pro_depth_rel_rgb_py} 0" rpy="0 0 0" />
+      <parent link="camera_rgb_frame" />
+      <child link="camera_depth_frame" />
+    </joint>
+    <link name="camera_depth_frame">
+      <inertial>
+        <mass value="0.01" />
+        <origin xyz="0 0 0" />
+        <inertia ixx="0.001" ixy="0.0" ixz="0.0"
+          iyy="0.001" iyz="0.0"
+          izz="0.001" />
+      </inertial>
+    </link>
+    <joint name="camera_depth_optical_joint" type="fixed">
+      <origin xyz="0 0 0" rpy="${-M_PI/2} 0 ${-M_PI/2}" />
+      <parent link="camera_depth_frame" />
+      <child link="camera_depth_optical_frame" />
+    </joint>
+    <link name="camera_depth_optical_frame">
+      <inertial>
+        <mass value="0.001" />
+        <origin xyz="0 0 0" />
+        <inertia ixx="0.0001" ixy="0.0" ixz="0.0"
+          iyy="0.0001" iyz="0.0"
+          izz="0.0001" />
+      </inertial>
+    </link>
+  <!-- RGBD sensor for simulation, same as Kinect -->
+  <turtlebot_sim_3dsensor/>
+  </xacro:macro>
 </robot>

File: gopherturtle_description/urdf/turtlebot_properties.urdf.xacro (robot description, xacro)
@@ -28,15 +28,15 @@
 	<!-- Front DSLAM cam -->
 	<property name="fcam_px" value="0.0806" />
-        <property name="fcam_py" value="0" />
-        <property name="fcam_pz" value="0.955" />
-        <property name="fcam_or" value="0" />
-        <property name="fcam_op" value="0" />
-        <property name="fcam_oy" value="0" />
+  <property name="fcam_py" value="0" />
+  <property name="fcam_pz" value="0.955" />
+  <property name="fcam_or" value="0" />
+  <property name="fcam_op" value="0" />
+  <property name="fcam_oy" value="0" />
 	<!-- Back DSLAM cam -->
 	<property name="bcam_px" value="-0.0806" />
-        <property name="bcam_py" value="0" />
-        <property name="bcam_pz" value="0.955" />
-        <property name="bcam_or" value="0" />
-        <property name="bcam_op" value="0" />
-        <property name="bcam_oy" value="0" />
+  <property name="bcam_py" value="0" />
+  <property name="bcam_pz" value="0.955" />
+  <property name="bcam_or" value="0" />
+  <property name="bcam_op" value="0" />
+  <property name="bcam_oy" value="3.14159265" />
 </robot>
